File: hardware/kicad/ac.kicad_sch (KiCad schematic)
At the start: 25 parts, among them J1 AC_Input, J2 Hirose RPC1-12RB-6P(71), Q1 KIA50N06BD, Q2 KIA50N06BD, U1 VOS628A, U2 L78L24_SOT89, U3 Si8751, U4 AP2111H-3.3

Commit message: [HW] Add: - Tag Connect Debug connector - USB & I2C breakout - GND pin to UART breakout
Parts:
- R1, R2, R3: footprint Resistor_SMD:R_0805_2012Metric -> Resistor_SMD:R_0603_1608Metric
Other:
- title: OpenSolder Station Schematic -> Marcs OpenSolder Station Schematic
