File: hardware/kicad/analog.kicad_sch (KiCad schematic)
At the start: 9 parts, among them U5 MAX4238ASA

Commit message: [HW] Add: - Tag Connect Debug connector - USB & I2C breakout - GND pin to UART breakout
Parts:
- C7, C8: footprint Capacitor_SMD:C_0805_2012Metric -> Capacitor_SMD:C_0603_1608Metric
- R4, R5, R6, R7: footprint Resistor_SMD:R_0805_2012Metric -> Resistor_SMD:R_0603_1608Metric
Other:
- title: OpenSolder Station Schematic -> Marcs OpenSolder Station Schematic
