File: hardware/kicad/opensolder.kicad_pcb (KiCad board)
At the start: 2 copper layers, 100 x 44 mm, 69 parts, among them J1 AC_Input, J2 Hirose RPC1-12RB-6P(71), J3 SWD, J4 UART, J5 Reset_Switch, Q1 KIA50N06BD, Q2 KIA50N06BD, SW2 PEC11R-RotEnc, U1 VOS628A, U2 L78L24_SOT89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

Commit message: [HW] Add: - Tag Connect Debug connector - USB & I2C breakout - GND pin to UART breakout
Parts:
- added C22: 100n, Capacitor_SMD:C_0603_1608Metric, F.Cu at (124.5, 115.6)
- added G***: LOGO, Logo:logo-30x9.8mm, B.Cu at (122.6, 102.9)
- added J6: Conn_ARM_SWD_TagConnect_TC2030-NL, Connector:Tag-Connect_TC2030-IDC-NL_2x03_P1.27mm_Vertical, F.Cu at (119.4, 92.7)
- added J7: USB, Connector_PinSocket_2.54mm:PinSocket_1x04_P2.54mm_Vertical, F.Cu at (122.6, 80.6)
- added R21: 3k3, Resistor_SMD:R_0603_1608Metric, F.Cu at (113.7, 85.7)
- added R22: 3k3, Resistor_SMD:R_0603_1608Metric, F.Cu at (109.2, 87.6)
- added R23: 3R3, Resistor_SMD:R_0603_1608Metric, F.Cu at (117.5, 84.5)
- added R24: 3R3, Resistor_SMD:R_0603_1608Metric, F.Cu at (120.0, 84.5)
- added R25: 10k, Resistor_SMD:R_0603_1608Metric, F.Cu at (124.5, 118.6)
- C10, C16, C17, C18, C19, C20, C21, C7, C8, C9: footprint Capacitor_SMD:C_0805_2012Metric -> Capacitor_SMD:C_0603_1608Metric
- J3: value SWD -> IO; footprint Connector_IDC:IDC-Header_2x03_P2.54mm_Vertical -> Connector_PinHeader_2.54mm:PinHeader_2x03_P2.54mm_Vertical
- J4: footprint Connector_PinSocket_2.54mm:PinSocket_1x02_P2.54mm_Vertical -> Connector_PinSocket_2.54mm:PinSocket_1x03_P2.54mm_Vertical
- R1, R10, R11, R12, R13, R14, R15, R16, R17, R18, R19, R2, R20, R3, R4, R5, R6, R7, R8, R9: footprint Resistor_SMD:R_0805_2012Metric -> Resistor_SMD:R_0603_1608Metric
- SW2: value PEC11R-RotEnc -> PEC11R-4220F-S0024
- moved J4 7.78 mm to (131.4, 80.6)
- moved J3 3.25 mm to (109.9, 81.9)
- moved J5 2.62 mm to (127.6, 115.6)
Connections:
- J3 pad 1: /MCU/SWCLK -> /MCU/I2C2_SCL
- J3 pad 2: /MCU/SWDIO -> /MCU/I2C2_SDA
- U7 pad 26: GND -> /MCU/I2C2_SCL
- U7 pad 27: GND -> /MCU/I2C2_SDA
- U7 pad 32: GND -> /MCU/USB_DN
- U7 pad 33: GND -> /MCU/USB_DP
Routing:
- net +5V: track 26.2 -> 67.7 mm, vias 0 -> 7
- net /MCU/NRST: track 16.6 -> 51.3 mm, vias 0 -> 2
- net /MCU/I2C2_SCL: track 0.00 -> 30.0 mm, vias 0 -> 2
- net /MCU/I2C2_SDA: track 0.00 -> 28.8 mm, vias 0 -> 4
- net /MCU/SWCLK: track 25.4 -> 7.25 mm, vias 2 -> 0
- net /MCU/USB_DP: track 0.00 -> 17.3 mm
- net /MCU/USB_DN: track 0.00 -> 16.2 mm
- net +3V3: track 209.6 -> 223.2 mm
- net /MCU/SWDIO: track 20.8 -> 10.1 mm, vias 0 -> 2
- net Net-(J7-Pin_3): track 0.00 -> 2.98 mm
- net Net-(J7-Pin_2): track 0.00 -> 2.98 mm
- net /MCU/UART_RX: track 16.8 -> 14.1 mm
- net GND: track 51.5 -> 48.9 mm, vias 260 -> 263
- net /MCU/STAND_CONN: track 40.6 -> 41.8 mm
- net /MCU/UART_TX: track 14.8 -> 15.8 mm
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Other:
- board text added: "+3V3"
- board text added: "5V DP DM +5V"
- board text added: "Designed: Håvard Jakobsen Modified: Marc Fischer"
- board text added: "GND"
- board text added: "GND Rx Tx"
- board text added: "OpenSolder"
- board text added: "SCL"
- board text added: "SDA"
- board text added: "STAND"
- board text added: "TIP"
- board text removed: "1: SWCLK 2: SWDIO 3: GND 4: +3V3 5: Tip Remover 6: Stand"
- board text removed: "5 3 1 6 4 2"
- board text removed: "Designer: Håvard Jakobsen"
- board text removed: "OpenSolder v1.0"
- board text removed: "Rx Tx"
