File: hardware/kicad/opensolder.kicad_sch (KiCad schematic)
At the start: 0 parts

Commit message: [HW] Add: - Tag Connect Debug connector - USB & I2C breakout - GND pin to UART breakout
Other:
- title: OpenSolder Station Schematic -> Marcs OpenSolder Station Schematic
